Commit message: upload local code

File: resources/robots/bolt10/urdf/bolt10.urdf (robot description, URDF)
Before this commit: robot bolt10_urdf, 11 links, 10 joints
Links:
- link L_Foot: geometry collision box size=0.10 0.03 0.02; visual mesh filename=../meshes/L_Foot_box.stl
- link R_Foot: geometry collision box size=0.10 0.03 0.02; visual mesh filename=../meshes/R_Foot_box.stl
- link base_link: mass 1.556324 -> 1.055; geometry collision sphere radius=0.15; visual mesh filename=../meshes/base_link_new.stl
Joints:
- joint L_AnklePitch_Joint: limit lower=-1.50 upper=1.50 effort=3.5 velocity=20 -> lower=-1.50 upper=1.50 effort=3.5 velocity=50
- joint L_HipPitch_Joint: limit lower=-1.57 upper=1.57 effort=4.4 velocity=20 -> lower=-1.57 upper=1.57 effort=4.4 velocity=50
- joint L_HipRoll_Joint: limit lower=-0.73 upper=1.57 effort=3.5 velocity=20 -> lower=-0.73 upper=1.57 effort=3.5 velocity=50
- joint L_HipYaw_Joint: limit lower=-0.43 upper=1.57 effort=3.5 velocity=20 -> lower=-0.43 upper=1.57 effort=3.5 velocity=50
- joint L_KneePitch_Joint: limit lower=0 upper=3.14 effort=4.4 velocity=20 -> lower=0 upper=3.14 effort=4.4 velocity=50
- joint R_AnklePitch_Joint: limit lower=-1.50 upper=1.50 effort=3.5 velocity=20 -> lower=-1.50 upper=1.50 effort=3.5 velocity=50
- joint R_HipPitch_Joint: limit lower=-1.57 upper=1.57 effort=4.4 velocity=20 -> lower=-1.57 upper=1.57 effort=4.4 velocity=50
- joint R_HipRoll_Joint: limit lower=-1.57 upper=0.73 effort=3.5 velocity=20 -> lower=-1.57 upper=0.73 effort=3.5 velocity=50
- joint R_HipYaw_Joint: limit lower=-1.57 upper=0.43 effort=3.5 velocity=20 -> lower=-1.57 upper=0.43 effort=3.5 velocity=50
- joint R_KneePitch_Joint: limit lower=0 upper=3.14 effort=4.4 velocity=20 -> lower=0 upper=3.14 effort=4.4 velocity=50

File: resources/robots/bolt6/urdf/bolt6.urdf (robot description, URDF)
Before this commit: robot bolt, 9 links, 8 joints
Joints:
- joint FL_ANKLE: limit lower=-1 upper=1 effort=2.5 velocity=20 -> lower=-1 upper=1 effort=2.5 velocity=50; origin xyz=0 0.008e -0.2 rpy=0 0 0 -> xyz=0 0.008 -0.2 rpy=0 0 0
- joint FL_HAA: limit lower=-0.36 upper=1.0472 effort=2.5 velocity=20 -> lower=-0.36 upper=1.0472 effort=2.5 velocity=50
- joint FL_HFE: limit lower=-1.57 upper=1.57 effort=2.5 velocity=20 -> lower=-1.57 upper=1.57 effort=2.5 velocity=50
- joint FL_KFE: limit lower=-0.0 upper=3.14 effort=2.5 velocity=20 -> lower=-3.14 upper=0.0 effort=2.5 velocity=50
- joint FR_ANKLE: limit lower=-1 upper=1 effort=2.5 velocity=20 -> lower=-1 upper=1 effort=2.5 velocity=50
- joint FR_HAA: limit lower=-1.0472 upper=0.36 effort=2.5 velocity=20 -> lower=-1.0472 upper=0.36 effort=2.5 velocity=50
- joint FR_HFE: limit lower=-1.57 upper=1.57 effort=2.5 velocity=20 -> lower=-1.57 upper=1.57 effort=2.5 velocity=50
- joint FR_KFE: limit lower=-0.0 upper=3.14 effort=2.5 velocity=20 -> lower=-3.14 upper=0.0 effort=2.5 velocity=50

Commit message: TOCABI walking still working

File: resources/robots/bolt10/urdf/bolt10.urdf (robot description, URDF)
Before this commit: robot bolt10_urdf, 11 links, 10 joints
Links:
- link base_link: geometry collision sphere radius=0.15; visual mesh filename=../meshes/base_link.stl

File: resources/robots/tocabi/urdf/tocabi.urdf (robot description, URDF)
Before this commit: robot tocabi, 37 links, 36 joints
Links:
- link Head_Link: geometry visual mesh filename=../meshes/head_v1.stl scale=0.001 0.001 0.001
- link L_Armlink_Link: geometry visual mesh filename=../meshes/L_arm.STL
- link L_Elbow_Link: geometry visual mesh filename=../meshes/L_elbow.STL
- link L_Forearm_Link: geometry visual mesh filename=../meshes/L_forearm.STL
- link L_Shoulder1_Link: geometry visual mesh filename=../meshes/L_shoulder1.STL
- link L_Shoulder2_Link: geometry visual mesh filename=../meshes/L_shoulder2.STL
- link L_Shoulder3_Link: geometry visual mesh filename=../meshes/L_shoulder3.STL
- link L_Wrist1_Link: geometry visual mesh filename=../meshes/L_wrist1.STL
- link L_Wrist2_Link: geometry visual box size=0.03 0.005 0.05; visual box size=0.03 0.005 0.05
- link Neck_Link: geometry visual mesh filename=../meshes/neck.STL
- link Pelvis_Link: geometry collision box size=0.141 0.305 0.35; visual mesh filename=../meshes/Pelvis_link.STL
- link R_Armlink_Link: geometry visual mesh filename=../meshes/R_arm.STL
- link R_Elbow_Link: geometry visual mesh filename=../meshes/R_elbow.STL
- link R_Forearm_Link: geometry visual mesh filename=../meshes/R_forearm.STL
- link R_Shoulder1_Link: geometry visual mesh filename=../meshes/R_shoulder1.STL
- link R_Shoulder2_Link: geometry visual mesh filename=../meshes/R_shoulder2.STL
- link R_Shoulder3_Link: geometry visual mesh filename=../meshes/R_shoulder3.STL
- link R_Wrist1_Link: geometry visual mesh filename=../meshes/R_wrist1.STL
- link R_Wrist2_Link: geometry visual box size=0.03 0.005 0.05; visual box size=0.03 0.005 0.05
- link Upperbody_Link: geometry visual box size=0.12 0.07 0.14; visual box size=0.21 0.11 0.07
- link Waist1_Link: geometry visual cylinder length=0.02 radius=0.05; visual mesh filename=../meshes/waist1.STL
- link Waist2_Link: geometry visual mesh filename=../meshes/waist2.STL
Joints:
- joint L_AnklePitch_Joint: limit lower=-1.047 upper=0.523 effort=500 velocity=12 -> lower=-1.047 upper=0.523 effort=300 velocity=12
- joint L_AnkleRoll_Joint: limit lower=-0.61 upper=0.61 effort=500 velocity=12 -> lower=-0.61 upper=0.61 effort=300 velocity=12
- joint L_Elbow_Joint: origin xyz=0 0.207 -0.0325 rpy=-1.57 0 0 -> xyz=0 0.207 -0.0325 rpy=0 0 0
- joint L_Knee_Joint: limit lower=0.09 upper=2.1 effort=500 velocity=12 -> lower=0.0 upper=2.1 effort=500 velocity=12
- joint R_AnklePitch_Joint: limit lower=-1.047 upper=0.523 effort=500 velocity=12 -> lower=-1.047 upper=0.523 effort=300 velocity=12
- joint R_AnkleRoll_Joint: limit lower=-0.61 upper=0.61 effort=500 velocity=12 -> lower=-0.61 upper=0.61 effort=300 velocity=12
- joint R_Elbow_Joint: origin xyz=0 -0.207 -0.0325 rpy=1.57 0 0 -> xyz=0 -0.207 -0.0325 rpy=0 0 0
- joint R_Knee_Joint: limit lower=0.09 upper=2.1 effort=500 velocity=12 -> lower=0.00 upper=2.1 effort=500 velocity=12
